File: Wind Sensor PCB/atmega328.kicad_sch (KiCad schematic)
At the start: 19 parts, among them P10 I2C, P3 ID, P4 ISP, P9 PROG, SW1 SWA, SW2 RST, U4 ATmega328P-AU, Y1 8MHz_XTAL

Commit message: Large update - firmware and PCB design. V2
Parts:
- R6, R7: value 10k -> 4k7; Manufacturer Part MC01W080554K7 -> 0805W8F4701T5E
Changed lines of the file:
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@@
 			)
 		)
-		(property "Value" "10k"
+		(property "Value" "4k7"
 			(at 207.01 76.2 90)
 			(effects
@@
 			)
 		)
-		(property "Manufacturer Part" "MC01W080554K7"
+		(property "Manufacturer Part" "0805W8F4701T5E"
 			(at 208.28 69.85 0)
 			(effects
@@
 		)
 		(property "JLCPCB Cost" "0.0031"
+			(at 208.28 69.85 0)
+			(effects
+				(font
+					(size 1.27 1.27)
+				)
+				(hide yes)
+			)
+		)
+		(property "Supplier 2" ""
+			(at 208.28 69.85 0)
+			(effects
+				(font
+					(size 1.27 1.27)
+				)
+				(hide yes)
+			)
+		)
+		(property "Supplier 2 Code" ""
+			(at 208.28 69.85 0)
+			(effects
+				(font
+					(size 1.27 1.27)
+				)
+				(hide yes)
+			)
+		)
+		(property "Supplier 2 Web" ""
+			(at 208.28 69.85 0)
+			(effects
+				(font
+					(size 1.27 1.27)
+				)
+				(hide yes)
+			)
+		)
+		(property "Manufacturer" ""
+			(at 208.28 69.85 0)
+			(effects
+				(font
+					(size 1.27 1.27)
+				)
+				(hide yes)
+			)
+		)
+		(property "Supplier 2 Cost" ""
 			(at 208.28 69.85 0)
 			(effects
@@
 			)
 		)
-		(property "Value" "10k"
+		(property "Value" "4k7"
 			(at 203.2 76.2 90)
 			(effects
@@
 			)
 		)
-		(property "Manufacturer Part" "MC01W080554K7"
+		(property "Manufacturer Part" "0805W8F4701T5E"
 			(at 204.47 69.85 0)
 			(effects
@@
 			(at 204.47 69.85 0)
 			(effects
+				(font
+					(size 1.27 1.27)
+				)
+				(hide yes)
+			)
+		)
+		(property "Supplier 2" ""
+			(at 204.47 69.85 0)
+			(effects
+				(font
+					(size 1.27 1.27)
+				)
+				(hide yes)
+			)
+		)
+		(property "Supplier 2 Code" ""
+			(at 204.47 69.85 0)
+			(effects
+				(font
+					(size 1.27 1.27)
+				)
+				(hide yes)
+			)
+		)
+		(property "Supplier 2 Web" ""
+			(at 204.47 69.85 0)
+			(effects
+				(font
+					(size 1.27 1.27)
+				)
+				(hide yes)
+			)
+		)
+		(property "Manufacturer" ""
+			(at 204.47 69.85 0)
+			(effects
+				(font
+					(size 1.27 1.27)
+				)
+				(hide yes)
+			)
+		)
+		(property "Supplier 2 Cost" ""
+			(at 204.47 69.85 0)
+			(effects
